File: Hardware/Laberinto prueba version 3.0/lab_V3.kicad_sch (KiCad schematic)
At the start: 27 parts, among them J1 MotorIzq, J10 DRV8833_IN, J11 DRV8833_OUT, J2 MotorDer, J3 SWITCH, J4 Jack_Batt, J5 Distancia_Izq, J6 Distancia_Frontal, J7 Distancia_Der, J8 Encoder_DER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

Commit message: continuamos PCB
Connections:
- net start is gone; now on net Start: U3.8 (IO25)
- net D1: now also U3.9 (IO26); no longer U3.10 (IO27)
- net Strategy_A: now also U3.10 (IO27); no longer U3.9 (IO26)
Other:
- moved on the sheet: C1, C2, C3, C4, Display1, H1, H2, J1, J10, J11, J2, J3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

Commit message: sch cambio
Parts:
- removed J1: MotorIzq, Connector_JST:JST_EH_B2B-EH-A_1x02_P2.50mm_Vertical, symbol Connector_Generic:Conn_01x02
- removed J2: MotorDer, Connector_JST:JST_EH_B2B-EH-A_1x02_P2.50mm_Vertical, symbol Connector_Generic:Conn_01x02
- removed J8: Encoder_DER, Connector_JST:JST_EH_B4B-EH-A_1x04_P2.50mm_Vertical, symbol Connector_Generic:Conn_01x04
- removed J9: Encoder_IZQ, Connector_JST:JST_EH_B4B-EH-A_1x04_P2.50mm_Vertical, symbol Connector_Generic:Conn_01x04
- added J?: Encoder Derecho, symbol EESTN5:Conn_01x06
- added J?: Encoder Izquierdo, symbol EESTN5:Conn_01x06
Connections:
- net +5V: now also J?.3 (Pin_3), J?.3 (Pin_3)
- net AOUT1: now also J?.1 (Pin_1)
- net AOUT2: now also J?.2 (Pin_2)
- net BOUT1: now also J?.2 (Pin_2)
- net BOUT2: now also J?.1 (Pin_1)
- net D1: now also U3.7 (IO33); no longer U3.9 (IO26)
- net GND: now also J?.6 (Pin_6), J?.6 (Pin_6)
- net IR_DER: now also U3.4 (IO34); no longer U3.6 (IO32)
- net IR_FRONTAL: now also U3.2 (SENSOR_VP); no longer U3.4 (IO34)
- net IR_IZQ: now also U3.3 (SENSOR_VN); no longer U3.5 (IO35)
- net Start: now also U3.6 (IO32); no longer U3.8 (IO25)
- net Strategy_A: now also U3.8 (IO25); no longer U3.10 (IO27)
- net TATAMI: now also U3.5 (IO35); no longer U3.7 (IO33)
- net D0 renamed D1A
- net D1A: now also U3.10 (IO27), J?.4 (Pin_4)
- new net D1B: J?.5 (Pin_5), U3.9 (IO26)
- new net D2A: J?.4 (Pin_4)
- new net D2B: J?.5 (Pin_5)
- no-connect marks 1 -> 11
Other:
- note added: "Houled Soporte Micro motores"
- note added: "Sensor Tatami"
- moved on the sheet: Display1, H1, H2, J3, J4, R2, R3, SW1, SW2, U2

Commit message: sch cambio2
Parts:
- removed SW2: SW_Push, EESTN5:Pulsador_TH_4, symbol EESTN5:SW_Push
- J1, J2: renamed from J?; footprint (none) -> EESTN5:pin_strip_6
Connections:
- net D1 is gone; now on net TATAMI: U3.7 (IO33)
- net Strategy_A is gone; now on net Start: U3.8 (IO25)
- net D1A: no longer U3.26 (IO21)
- net D2A: now also U3.26 (IO21)
- net IR_DER: now also U3.6 (IO32); no longer U3.4 (IO34)
- net IR_FRONTAL: now also U3.4 (IO34); no longer U3.2 (SENSOR_VP)
- net IR_IZQ: now also U3.5 (IO35); no longer U3.3 (SENSOR_VN)
- net Start: no longer U3.6 (IO32)
- net TATAMI: no longer U3.5 (IO35)
Other:
- moved on the sheet: J7, SW1
