File: Hardware/Laberinto prueba version 3.0/lab_V3.kicad_sch (KiCad schematic)
At the start: 24 parts, among them J1 Encoder Derecho, J10 DRV8833_IN, J11 DRV8833_OUT, J2 Encoder Izquierdo, J3 SWITCH, J4 Jack_Batt, J5 Distancia_Izq, J6 Distancia_Frontal, J7 Distancia_Der, SW1 SW_Push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

Commit message: estamos haciendo la placa ya
Parts:
- renumbered SW1 to Start1
Other:
- moved on the sheet: J10, J11

Commit message: cambios en el diseño 3d de soportes IR
Parts:
- C1: value 220uF -> (none); footprint EESTN5:C_1206 -> (none)
- C3: value 10uF -> (none); footprint EESTN5:C_1206 -> (none)
Connections:
- net +5V: now also Start1.1
- net GND: no longer Start1.1
Changed lines of the file:
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@@
     (stroke (width 0) (type default) (color 0 0 0 0))
   )
-  (wire (pts (xy 41.2496 24.1554) (xy 41.2496 25.9334))
-    (stroke (width 0) (type default) (color 0 0 0 0))
-  )
   (wire (pts (xy 30.1752 71.7804) (xy 30.1752 64.3128))
     (stroke (width 0) (type default) (color 0 0 0 0))
@@
       (effects (font (size 1.27 1.27)) (justify left))
     )
-    (property "Value" "220uF" (id 1) (at 17.9832 107.9754 0)
+    (property "Value" "" (id 1) (at 17.9832 107.9754 0)
       (effects (font (size 1.27 1.27)) (justify left))
     )
-    (property "Footprint" "EESTN5:C_1206" (id 2) (at 25.9842 107.2388 0)
+    (property "Footprint" "" (id 2) (at 25.9842 107.2388 0)
       (effects (font (size 1.27 1.27)) hide)
     )
@@
       (effects (font (size 1.27 1.27)) (justify left))
     )
-    (property "Value" "10uF" (id 1) (at 50.3682 108.1024 0)
+    (property "Value" "" (id 1) (at 50.3682 108.1024 0)
       (effects (font (size 1.27 1.27)) (justify left))
     )
-    (property "Footprint" "EESTN5:C_1206" (id 2) (at 56.6166 106.172 0)
+    (property "Footprint" "" (id 2) (at 56.6166 106.172 0)
       (effects (font (size 1.27 1.27)) hide)
     )
@@
     (pin "1")
   )
-  (symbol (lib_id "power:GND") (at 41.2496 25.9334 0) (unit 1)
-    (in_bom yes) (on_board yes) (fields_autoplaced)
-    (property "Reference" "#PWR02" (id 0) (at 41.2496 32.2834 0)
-      (effects (font (size 1.27 1.27)) hide)
-    )
-    (property "Value" "GND" (id 1) (at 41.2496 31.5214 0))
-    (property "Footprint" "" (id 2) (at 41.2496 25.9334 0)
-      (effects (font (size 1.27 1.27)) hide)
-    )
-    (property "Datasheet" "" (id 3) (at 41.2496 25.9334 0)
-      (effects (font (size 1.27 1.27)) hide)
-    )
-    (pin "1")
-  )
   (symbol (lib_id "power:GND") (at 38.0492 75.946 0) (unit 1)
     (in_bom yes) (on_board yes) (fields_autoplaced)
@@
     (pin "1")
   )
+  (symbol (lib_id "power:+5V") (at 41.2496 24.1554 0) (unit 1)
+    (in_bom yes) (on_board yes)
+    (property "Reference" "#PWR0105" (id 0) (at 41.2496 27.9654 0)
+      (effects (font (size 1.27 1.27)) hide)
+    )
+    (property "Value" "+5V" (id 1) (at 41.3766 20.7264 0))
+    (property "Footprint" "" (id 2) (at 41.2496 24.1554 0)
+      (effects (font (size 1.27 1.27)) hide)
+    )
+    (property "Datasheet" "" (id 3) (at 41.2496 24.1554 0)
+      (effects (font (size 1.27 1.27)) hide)
+    )
+    (pin "1")
+  )
   (symbol (lib_id "Connector_Generic:Conn_01x03") (at 194.945 66.0908 0) (unit 1)
     (in_bom yes) (on_board yes) (fields_autoplaced)
@@
       (reference "#PWR01") (unit 1) (value "+BATT") (footprint "")
     )
-    (path "/d3d9c44c-4a9d-4d68-a80d-d4c84e8a97e8"
-      (reference "#PWR02") (unit 1) (value "GND") (footprint "")
-    )
     (path "/5cece541-f5f1-420f-8059-847a13ee05fb"
       (reference "#PWR04") (unit 1) (value "GND") (footprint "")
@@
       (reference "#PWR0104") (unit 1) (value "+5V") (footprint "")
     )
+    (path "/e6c82ad4-5cf4-43ca-a7bb-9ff08ef84d94"
+      (reference "#PWR0105") (unit 1) (value "+5V") (footprint "")
+    )
     (path "/6cd21d84-b46b-4ae6-aecb-f2e0d6c78348"
-      (reference "C1") (unit 1) (value "220uF") (footprint "EESTN5:C_1206")
+      (reference "C1") (unit 1) (value "220uF") (footprint "EESTN5:CAP_ELEC_5x11mm")
     )
     (path "/c0904fde-1e50-44fa-8bc5-852691ceacef"
@@
     )
     (path "/84050798-b48e-4a26-974f-71e48e6d0cbb"
-      (reference "C3") (unit 1) (value "10uF") (footprint "EESTN5:C_1206")
+      (reference "C3") (unit 1) (value "220uF") (footprint "EESTN5:CAP_ELEC_5x11mm")
     )
     (path "/393a40e0-3cb5-4079-b2e6-9e2aa34aca5e"
