File: Hardware/Laberinto prueba version 3.0/lab_V3 (Copia en conflicto de LEANDRO BENÍTEZ 2022-09-19).kicad_sch (KiCad schematic)
At the start: 24 parts, among them J1 Encoder Derecho, J10 DRV8833_IN, J11 DRV8833_OUT, J2 Encoder Izquierdo, J3 SWITCH, J4 Jack_Batt, J5 Distancia_Izq, J6 Distancia_Frontal, J7 Distancia_Der, SW1 SW_Push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

Commit message: Placa lista solo faltan alguna correcciones de taiel
Parts:
- J1, J2: footprint Connector_JST:JST_EH_B6B-EH-A_1x06_P2.50mm_Vertical -> EESTN5:pin_strip_6
- LED1: footprint EESTN5:led_5mm_green -> EESTN5:LED_1206
Connections:
- net AIN1: now also U3.24 (IO18); no longer U3.25 (IO19)
- net AIN2: now also U3.25 (IO19); no longer U3.24 (IO18)
- net AOUT1: now also J11.5 (Pin_5); no longer J11.3 (Pin_3)
- net AOUT2: now also J11.4 (Pin_4); no longer J11.2 (Pin_2)
- net BOUT1: now also J11.2 (Pin_2), J2.2 (Pin_2); no longer J11.4 (Pin_4), J2.1 (Pin_1)
- net BOUT2: now also J11.3 (Pin_3), J2.1 (Pin_1); no longer J11.5 (Pin_5), J2.2 (Pin_2)
- net D2B: now also U3.10 (IO27); no longer U3.7 (IO33)
- net IR_DER: now also U3.5 (IO35); no longer U3.10 (IO27)
- net IR_FRONTAL: now also U3.6 (IO32); no longer U3.5 (IO35)
- net TATAMI: now also U3.7 (IO33); no longer U3.6 (IO32)
Other:
- moved on the sheet: J3, J4
